Commit message: added new urdf and added colour on links

File: urdf/materials.xacro (robot description, xacro)
@@ -2,5 +2,21 @@
 <robot name="mr_robot" xmlns:xacro="http://www.ros.org/wiki/xacro" >
 <material name="silver">
-  <color rgba="0.700 0.700 0.700 1.000"/>
+  <color rgba="0.700 0.740 0.700 1.000"/>
+</material>
+<material name="translucent">
+  <color rgba="0.27 0.33 0.3 0.5"/>
+  <phong>
+    <specular>1</specular>
+    <shininess>100</shininess>
+  </phong>
+</material>
+<material name="black">
+  <color rgba="0 0 0 1"/>
+</material>
+<material name="dark_grey">
+  <color rgba="0.24 0.26 0.24 1"/>
+</material>
+<material name="blue">
+  <color rgba="0 0 1 1"/>
 </material>
 </robot>

File: urdf/mr_robot.xacro (robot description, xacro)
@@ -26,5 +26,5 @@
 <link name="tyre_r_1">
   <inertial>
-    <origin xyz="0.06525409087830025 -7.085638543073307e-06 -0.0009998838120615534" rpy="0 0 0"/>
+    <origin xyz="0.06525409087830011 -7.03390812247892e-06 -0.0010000781645711151" rpy="0 0 0"/>
     <mass value="2.445514992570597"/>
     <inertia ixx="0.00501" iyy="0.003032" izz="0.003032" ixy="0.0" iyz="0.0" ixz="0.0"/>
@@ -35,5 +35,5 @@
       <mesh filename="package://mr_robot_description/meshes/tyre_r_1.stl" scale="0.001 0.001 0.001"/>
     </geometry>
-    <material name="silver"/>
+    <material name="black"/>
   </visual>
   <collision>
@@ -55,5 +55,5 @@
       <mesh filename="package://mr_robot_description/meshes/tyre_l_1.stl" scale="0.001 0.001 0.001"/>
     </geometry>
-    <material name="silver"/>
+    <material name="black"/>
   </visual>
   <collision>
@@ -75,5 +75,5 @@
       <mesh filename="package://mr_robot_description/meshes/lidar_1.stl" scale="0.001 0.001 0.001"/>
     </geometry>
-    <material name="silver"/>
+    <material name="blue"/>
   </visual>
   <collision>
@@ -81,4 +81,44 @@
     <geometry>
       <mesh filename="package://mr_robot_description/meshes/lidar_1.stl" scale="0.001 0.001 0.001"/>
+    </geometry>
+  </collision>
+</link>
+<link name="upper_panel_1">
+  <inertial>
+    <origin xyz="-0.18750361570760787 -0.169810681160802 0.01845928081380513" rpy="0 0 0"/>
+    <mass value="7.649753398983407"/>
+    <inertia ixx="0.097265" iyy="0.111429" izz="0.205922" ixy="-1.5e-05" iyz="0.001292" ixz="5e-06"/>
+  </inertial>
+  <visual>
+    <origin xyz="-0.187549 -0.187451 -0.074" rpy="0 0 0"/>
+    <geometry>
+      <mesh filename="package://mr_robot_description/meshes/upper_panel_1.stl" scale="0.001 0.001 0.001"/>
+    </geometry>
+    <material name="translucent"/>
+  </visual>
+  <collision>
+    <origin xyz="-0.187549 -0.187451 -0.074" rpy="0 0 0"/>
+    <geometry>
+      <mesh filename="package://mr_robot_description/meshes/upper_panel_1.stl" scale="0.001 0.001 0.001"/>
+    </geometry>
+  </collision>
+</link>
+<link name="V_Slot_1">
+  <inertial>
+    <origin xyz="-0.1901793582234545 -0.14650407539123805 0.010262998829977818" rpy="0 0 0"/>
+    <mass value="1.4085607585669755"/>
+    <inertia ixx="0.015757" iyy="0.005506" izz="0.021181" ixy="2.8e-05" iyz="-1.3e-05" ixz="0.0"/>
+  </inertial>
+  <visual>
+    <origin xyz="-0.189955 -0.189958 -0.108" rpy="0 0 0"/>
+    <geometry>
+      <mesh filename="package://mr_robot_description/meshes/V_Slot_1.stl" scale="0.001 0.001 0.001"/>
+    </geometry>
+    <material name="dark_grey"/>
+  </visual>
+  <collision>
+    <origin xyz="-0.189955 -0.189958 -0.108" rpy="0 0 0"/>
+    <geometry>
+      <mesh filename="package://mr_robot_description/meshes/V_Slot_1.stl" scale="0.001 0.001 0.001"/>
     </geometry>
   </collision>
@@ -101,3 +141,13 @@
   <child link="lidar_1"/>
 </joint>
+<joint name="Rigid 13" type="fixed">
+  <origin xyz="0.187549 0.187451 0.074" rpy="0 0 0"/>
+  <parent link="base_link"/>
+  <child link="upper_panel_1"/>
+</joint>
+<joint name="Rigid 14" type="fixed">
+  <origin xyz="0.002406 0.002507 0.034" rpy="0 0 0"/>
+  <parent link="upper_panel_1"/>
+  <child link="V_Slot_1"/>
+</joint>
 </robot>

Commit message: added more color in links

File: urdf/materials.xacro (robot description, xacro)
@@ -6,8 +6,4 @@
 <material name="translucent">
   <color rgba="0.27 0.33 0.3 0.5"/>
-  <phong>
-    <specular>1</specular>
-    <shininess>100</shininess>
-  </phong>
 </material>
 <material name="black">
@@ -20,3 +16,18 @@
   <color rgba="0 0 1 1"/>
 </material>
+<material name="orange">
+  <color rgba="0.8 0.35 0.10  1"/>
+</material>
+<material name="red">
+  <color rgba="1 0 0 1"/>
+</material>
+<material name="green">
+  <color rgba="0.08 0.6 0.21 1"/>
+</material>
+<material name="dark_red">
+  <color rgba="1 0.08 0.2 1"/>
+</material>
+<material name="white">
+  <color rgba="1 1 1  1"/>
+</material>
 </robot>

File: urdf/mr_robot.xacro (robot description, xacro)
@@ -35,5 +35,5 @@
       <mesh filename="package://mr_robot_description/meshes/tyre_r_1.stl" scale="0.001 0.001 0.001"/>
     </geometry>
-    <material name="silver"/>
+    <material name="black"/>
   </visual>
   <collision>
@@ -55,5 +55,5 @@
       <mesh filename="package://mr_robot_description/meshes/tyre_l_1.stl" scale="0.001 0.001 0.001"/>
     </geometry>
-    <material name="silver"/>
+    <material name="black"/>
   </visual>
   <collision>
@@ -71,12 +71,12 @@
   </inertial>
   <visual>
-    <origin xyz="9.4e-05 -0.183507 -0.005" rpy="0 0 0"/>
+    <origin xyz="9.4e-05 -0.104 -0.085" rpy="0 0 0"/>
     <geometry>
       <mesh filename="package://mr_robot_description/meshes/lidar_1.stl" scale="0.001 0.001 0.001"/>
     </geometry>
-    <material name="silver"/>
-  </visual>
-  <collision>
-    <origin xyz="9.4e-05 -0.183507 -0.005" rpy="0 0 0"/>
+    <material name="blue"/>
+  </visual>
+  <collision>
+    <origin xyz="9.4e-05 -0.104 -0.085" rpy="0 0 0"/>
     <geometry>
       <mesh filename="package://mr_robot_description/meshes/lidar_1.stl" scale="0.001 0.001 0.001"/>
@@ -95,5 +95,5 @@
       <mesh filename="package://mr_robot_description/meshes/upper_panel_1.stl" scale="0.001 0.001 0.001"/>
     </geometry>
-    <material name="silver"/>
+    <material name="translucent"/>
   </visual>
   <collision>
@@ -115,5 +115,5 @@
       <mesh filename="package://mr_robot_description/meshes/V_Slot_1.stl" scale="0.001 0.001 0.001"/>
     </geometry>
-    <material name="silver"/>
+    <material name="dark_grey"/>
   </visual>
   <collision>
@@ -135,5 +135,5 @@
       <mesh filename="package://mr_robot_description/meshes/RPi4ModelB_1.stl" scale="0.001 0.001 0.001"/>
     </geometry>
-    <material name="silver"/>
+    <material name="green"/>
   </visual>
   <collision>
@@ -155,5 +155,5 @@
       <mesh filename="package://mr_robot_description/meshes/LiPo_3S_v2_1.stl" scale="0.001 0.001 0.001"/>
     </geometry>
-    <material name="silver"/>
+    <material name="orange"/>
   </visual>
   <collision>
@@ -175,5 +175,5 @@
       <mesh filename="package://mr_robot_description/meshes/PCB_1_1.stl" scale="0.001 0.001 0.001"/>
     </geometry>
-    <material name="silver"/>
+    <material name="red"/>
   </visual>
   <collision>
@@ -195,5 +195,5 @@
       <mesh filename="package://mr_robot_description/meshes/motor_driver_1.stl" scale="0.001 0.001 0.001"/>
     </geometry>
-    <material name="silver"/>
+    <material name="dark_red"/>
   </visual>
   <collision>
@@ -215,5 +215,5 @@
       <mesh filename="package://mr_robot_description/meshes/PCB__1.stl" scale="0.001 0.001 0.001"/>
     </geometry>
-    <material name="silver"/>
+    <material name="red"/>
   </visual>
   <collision>
@@ -235,5 +235,5 @@
       <mesh filename="package://mr_robot_description/meshes/atom_1.stl" scale="0.001 0.001 0.001"/>
     </geometry>
-    <material name="silver"/>
+    <material name="white"/>
   </visual>
   <collision>
@@ -255,5 +255,5 @@
       <mesh filename="package://mr_robot_description/meshes/robotics_1.stl" scale="0.001 0.001 0.001"/>
     </geometry>
-    <material name="silver"/>
+    <material name="white"/>
   </visual>
   <collision>
@@ -268,5 +268,5 @@
   <parent link="base_link"/>
   <child link="tyre_r_1"/>
-  <axis xyz="1.0 -0.0 -0.0"/>
+  <axis xyz="-1.0 -0.0 -0.0"/>
 </joint>
 <joint name="Revolute 10" type="continuous">
@@ -277,5 +277,5 @@
 </joint>
 <joint name="Rigid 11" type="fixed">
-  <origin xyz="-9.4e-05 0.183507 0.005" rpy="0 0 0"/>
+  <origin xyz="-9.4e-05 0.104 0.09" rpy="0 0 0"/>
   <parent link="base_link"/>
   <child link="lidar_1"/>
