Commit message: fix lidar tf

File: urdf/mr_robot.xacro (robot description, xacro)
@@ -71,5 +71,5 @@
   </inertial>
   <visual>
-    <origin xyz="9.4e-05 -0.183507 -0.005" rpy="0 0 0"/>
+    <origin xyz="9.4e-05 -0.104 -0.085" rpy="0 0 0"/>
     <geometry>
       <mesh filename="package://mr_robot_description/meshes/lidar_1.stl" scale="0.001 0.001 0.001"/>
@@ -78,5 +78,5 @@
   </visual>
   <collision>
-    <origin xyz="9.4e-05 -0.183507 -0.005" rpy="0 0 0"/>
+    <origin xyz="9.4e-05 -0.104 -0.085" rpy="0 0 0"/>
     <geometry>
       <mesh filename="package://mr_robot_description/meshes/lidar_1.stl" scale="0.001 0.001 0.001"/>
@@ -97,5 +97,5 @@
 </joint>
 <joint name="Rigid 11" type="fixed">
-  <origin xyz="-9.4e-05 0.183507 0.005" rpy="0 0 0"/>
+  <origin xyz="-9.4e-05 0.104 0.09" rpy="0 0 0"/>
   <parent link="base_link"/>
   <child link="lidar_1"/>

Commit message: added pi, lipo, atom

File: urdf/mr_robot.xacro (robot description, xacro)
@@ -35,5 +35,5 @@
       <mesh filename="package://mr_robot_description/meshes/tyre_r_1.stl" scale="0.001 0.001 0.001"/>
     </geometry>
-    <material name="black"/>
+    <material name="silver"/>
   </visual>
   <collision>
@@ -55,5 +55,5 @@
       <mesh filename="package://mr_robot_description/meshes/tyre_l_1.stl" scale="0.001 0.001 0.001"/>
     </geometry>
-    <material name="black"/>
+    <material name="silver"/>
   </visual>
   <collision>
@@ -71,12 +71,12 @@
   </inertial>
   <visual>
-    <origin xyz="9.4e-05 -0.104 -0.085" rpy="0 0 0"/>
+    <origin xyz="9.4e-05 -0.183507 -0.005" rpy="0 0 0"/>
     <geometry>
       <mesh filename="package://mr_robot_description/meshes/lidar_1.stl" scale="0.001 0.001 0.001"/>
     </geometry>
-    <material name="blue"/>
-  </visual>
-  <collision>
-    <origin xyz="9.4e-05 -0.104 -0.085" rpy="0 0 0"/>
+    <material name="silver"/>
+  </visual>
+  <collision>
+    <origin xyz="9.4e-05 -0.183507 -0.005" rpy="0 0 0"/>
     <geometry>
       <mesh filename="package://mr_robot_description/meshes/lidar_1.stl" scale="0.001 0.001 0.001"/>
@@ -95,5 +95,5 @@
       <mesh filename="package://mr_robot_description/meshes/upper_panel_1.stl" scale="0.001 0.001 0.001"/>
     </geometry>
-    <material name="translucent"/>
+    <material name="silver"/>
   </visual>
   <collision>
@@ -106,7 +106,7 @@
 <link name="V_Slot_1">
   <inertial>
-    <origin xyz="-0.1901793582234545 -0.14650407539123805 0.010262998829977818" rpy="0 0 0"/>
-    <mass value="1.4085607585669755"/>
-    <inertia ixx="0.015757" iyy="0.005506" izz="0.021181" ixy="2.8e-05" iyz="-1.3e-05" ixz="0.0"/>
+    <origin xyz="-0.18995499999999968 -0.1874580000000005 0.010160324118212424" rpy="0 0 0"/>
+    <mass value="0.9613817576893362"/>
+    <inertia ixx="0.010478" iyy="0.004833" izz="0.015232" ixy="-0.0" iyz="0.0" ixz="-0.0"/>
   </inertial>
   <visual>
@@ -115,5 +115,5 @@
       <mesh filename="package://mr_robot_description/meshes/V_Slot_1.stl" scale="0.001 0.001 0.001"/>
     </geometry>
-    <material name="dark_grey"/>
+    <material name="silver"/>
   </visual>
   <collision>
@@ -121,4 +121,144 @@
     <geometry>
       <mesh filename="package://mr_robot_description/meshes/V_Slot_1.stl" scale="0.001 0.001 0.001"/>
+    </geometry>
+  </collision>
+</link>
+<link name="RPi4ModelB_1">
+  <inertial>
+    <origin xyz="0.01457205025824198 -0.07941383200423409 0.004004061740386505" rpy="0 0 0"/>
+    <mass value="0.043638650995952065"/>
+    <inertia ixx="1.3e-05" iyy="3e-05" izz="4e-05" ixy="0.0" iyz="0.0" ixz="-3e-06"/>
+  </inertial>
+  <visual>
+    <origin xyz="-4e-06 -0.009908 -0.078" rpy="0 0 0"/>
+    <geometry>
+      <mesh filename="package://mr_robot_description/meshes/RPi4ModelB_1.stl" scale="0.001 0.001 0.001"/>
+    </geometry>
+    <material name="silver"/>
+  </visual>
+  <collision>
+    <origin xyz="-4e-06 -0.009908 -0.078" rpy="0 0 0"/>
+    <geometry>
+      <mesh filename="package://mr_robot_description/meshes/RPi4ModelB_1.stl" scale="0.001 0.001 0.001"/>
+    </geometry>
+  </collision>
+</link>
+<link name="LiPo_3S_v2_1">
+  <inertial>
+    <origin xyz="0.04000862047942958 0.039993000000002554 0.021424999999999812" rpy="0 0 0"/>
+    <mass value="1.1316523601774637"/>
+    <inertia ixx="0.000601" iyy="0.004185" izz="0.004409" ixy="0.0" iyz="0.0" ixz="0.0"/>
+  </inertial>
+  <visual>
+    <origin xyz="9.4e-05 0.172993 -0.005" rpy="0 0 0"/>
+    <geometry>
+      <mesh filename="package://mr_robot_description/meshes/LiPo_3S_v2_1.stl" scale="0.001 0.001 0.001"/>
+    </geometry>
+    <material name="silver"/>
+  </visual>
+  <collision>
+    <origin xyz="9.4e-05 0.172993 -0.005" rpy="0 0 0"/>
+    <geometry>
+      <mesh filename="package://mr_robot_description/meshes/LiPo_3S_v2_1.stl" scale="0.001 0.001 0.001"/>
+    </geometry>
+  </collision>
+</link>
+<link name="PCB_1_1">
+  <inertial>
+    <origin xyz="-0.054883976883169205 -0.039951135342914834 0.009799999999999379" rpy="0 0 0"/>
+    <mass value="0.09316520405438372"/>
+    <inertia ixx="4.1e-05" iyy="8.2e-05" izz="0.000123" ixy="-0.0" iyz="-0.0" ixz="0.0"/>
+  </inertial>
+  <visual>
+    <origin xyz="-0.159906 -0.150007 -0.005" rpy="0 0 0"/>
+    <geometry>
+      <mesh filename="package://mr_robot_description/meshes/PCB_1_1.stl" scale="0.001 0.001 0.001"/>
+    </geometry>
+    <material name="silver"/>
+  </visual>
+  <collision>
+    <origin xyz="-0.159906 -0.150007 -0.005" rpy="0 0 0"/>
+    <geometry>
+      <mesh filename="package://mr_robot_description/meshes/PCB_1_1.stl" scale="0.001 0.001 0.001"/>
+    </geometry>
+  </collision>
+</link>
+<link name="motor_driver_1">
+  <inertial>
+    <origin xyz="0.0003955010685046656 0.0021371126752723303 0.006441770608912843" rpy="0 0 0"/>
+    <mass value="0.05766626670761933"/>
+    <inertia ixx="1.2e-05" iyy="9e-06" izz="1.5e-05" ixy="0.0" iyz="-2e-06" ixz="0.0"/>
+  </inertial>
+  <visual>
+    <origin xyz="0.0 0.0 -0.004" rpy="0 0 0"/>
+    <geometry>
+      <mesh filename="package://mr_robot_description/meshes/motor_driver_1.stl" scale="0.001 0.001 0.001"/>
+    </geometry>
+    <material name="silver"/>
+  </visual>
+  <collision>
+    <origin xyz="0.0 0.0 -0.004" rpy="0 0 0"/>
+    <geometry>
+      <mesh filename="package://mr_robot_description/meshes/motor_driver_1.stl" scale="0.001 0.001 0.001"/>
+    </geometry>
+  </collision>
+</link>
+<link name="PCB__1">
+  <inertial>
+    <origin xyz="0.06152156956597747 -0.04641560143698002 0.00980000000000017" rpy="0 0 0"/>
+    <mass value="0.09316520405438372"/>
+    <inertia ixx="4.1e-05" iyy="8.2e-05" izz="0.000123" ixy="-0.0" iyz="-0.0" ixz="0.0"/>
+  </inertial>
+  <visual>
+    <origin xyz="0.150094 -0.160007 -0.005" rpy="0 0 0"/>
+    <geometry>
+      <mesh filename="package://mr_robot_description/meshes/PCB__1.stl" scale="0.001 0.001 0.001"/>
+    </geometry>
+    <material name="silver"/>
+  </visual>
+  <collision>
+    <origin xyz="0.150094 -0.160007 -0.005" rpy="0 0 0"/>
+    <geometry>
+      <mesh filename="package://mr_robot_description/meshes/PCB__1.stl" scale="0.001 0.001 0.001"/>
+    </geometry>
+  </collision>
+</link>
+<link name="atom_1">
+  <inertial>
+    <origin xyz="0.0025939999999966823 0.014044204860724581 -0.0013535283083131039" rpy="0 0 0"/>
+    <mass value="0.20117543498961754"/>
+    <inertia ixx="0.001282" iyy="4.6e-05" izz="0.001236" ixy="-0.0" iyz="-9e-06" ixz="-0.0"/>
+  </inertial>
+  <visual>
+    <origin xyz="-0.176906 -7e-06 -0.04" rpy="0 0 0"/>
+    <geometry>
+      <mesh filename="package://mr_robot_description/meshes/atom_1.stl" scale="0.001 0.001 0.001"/>
+    </geometry>
+    <material name="silver"/>
+  </visual>
+  <collision>
+    <origin xyz="-0.176906 -7e-06 -0.04" rpy="0 0 0"/>
+    <geometry>
+      <mesh filename="package://mr_robot_description/meshes/atom_1.stl" scale="0.001 0.001 0.001"/>
+    </geometry>
+  </collision>
+</link>
+<link name="robotics_1">
+  <inertial>
+    <origin xyz="-0.002499999999996838 0.003416208393034576 0.0006064156437464094" rpy="0 0 0"/>
+    <mass value="0.2187386210217494"/>
+    <inertia ixx="0.001656" iyy="3.3e-05" izz="0.001624" ixy="0.0" iyz="-3e-06" ixz="0.0"/>
+  </inertial>
+  <visual>
+    <origin xyz="0.177 0.0 -0.039" rpy="0 0 0"/>
+    <geometry>
+      <mesh filename="package://mr_robot_description/meshes/robotics_1.stl" scale="0.001 0.001 0.001"/>
+    </geometry>
+    <material name="silver"/>
+  </visual>
+  <collision>
+    <origin xyz="0.177 0.0 -0.039" rpy="0 0 0"/>
+    <geometry>
+      <mesh filename="package://mr_robot_description/meshes/robotics_1.stl" scale="0.001 0.001 0.001"/>
     </geometry>
   </collision>
@@ -128,5 +268,5 @@
   <parent link="base_link"/>
   <child link="tyre_r_1"/>
-  <axis xyz="-1.0 -0.0 -0.0"/>
+  <axis xyz="1.0 -0.0 -0.0"/>
 </joint>
 <joint name="Revolute 10" type="continuous">
@@ -137,5 +277,5 @@
 </joint>
 <joint name="Rigid 11" type="fixed">
-  <origin xyz="-9.4e-05 0.104 0.09" rpy="0 0 0"/>
+  <origin xyz="-9.4e-05 0.183507 0.005" rpy="0 0 0"/>
   <parent link="base_link"/>
   <child link="lidar_1"/>
@@ -151,3 +291,38 @@
   <child link="V_Slot_1"/>
 </joint>
+<joint name="Rigid 15" type="fixed">
+  <origin xyz="-0.187545 -0.177543 0.004" rpy="0 0 0"/>
+  <parent link="upper_panel_1"/>
+  <child link="RPi4ModelB_1"/>
+</joint>
+<joint name="Rigid 16" type="fixed">
+  <origin xyz="-9.4e-05 -0.172993 0.005" rpy="0 0 0"/>
+  <parent link="base_link"/>
+  <child link="LiPo_3S_v2_1"/>
+</joint>
+<joint name="Rigid 17" type="fixed">
+  <origin xyz="0.159906 0.150007 0.005" rpy="0 0 0"/>
+  <parent link="base_link"/>
+  <child link="PCB_1_1"/>
+</joint>
+<joint name="Rigid 18" type="fixed">
+  <origin xyz="0.0 0.0 0.004" rpy="0 0 0"/>
+  <parent link="base_link"/>
+  <child link="motor_driver_1"/>
+</joint>
+<joint name="Rigid 19" type="fixed">
+  <origin xyz="-0.150094 0.160007 0.005" rpy="0 0 0"/>
+  <parent link="base_link"/>
+  <child link="PCB__1"/>
+</joint>
+<joint name="Rigid 20" type="fixed">
+  <origin xyz="0.176906 7e-06 0.04" rpy="0 0 0"/>
+  <parent link="base_link"/>
+  <child link="atom_1"/>
+</joint>
+<joint name="Rigid 21" type="fixed">
+  <origin xyz="-0.177 0.0 0.039" rpy="0 0 0"/>
+  <parent link="base_link"/>
+  <child link="robotics_1"/>
+</joint>
 </robot>
